File: CAN_Isolation/CAN_Isolation.kicad_pcb (KiCad board)
At the start: 4 copper layers, 120 x 60 mm, 61 parts, among them J1 S4B-XH-A, J10 Conn_01x28, J11 Conn_01x28, J12 Conn_01x28, J13 Conn_01x28, J14 Conn_01x28, J15 Conn_01x28, J16 Conn_01x28, J17 Conn_01x28, J2 Conn_01x28, J3 Conn_01x28, J4 Conn_01x28, J5 Conn_01x28, J6 Conn_01x28, J7 Conn_01x28, J8 Conn_01x28, J9 Conn_01x28, U1 MCP2518FDT-H/SL, U2 ISO1042QDWVRQ1, U3 MGS3123R3, U4 MGS1R51205, U5 TVS1800DRVR, U6 DTC114ECAHZGT116, U7 TPS610333QDRLRQ1, Y1 CSTNE20M0V530000R0

Commit message: Change board size.
Change board size.
Parts:
- moved G*** 5.48 mm to (169.5, 72.5)
- moved REF** 5.00 mm to (143.7, 72.8)
- moved REF** 5.00 mm to (143.7, 122.8)
Routing:
- net RF_GND: track 296.0 -> 294.7 mm
Changed lines of the file:
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@@
 	(footprint "MountingHole:MountingHole_3.2mm_M3"
 		(layer "F.Cu")
-		(at 148.657095 72.794905)
+		(at 143.657095 72.794905)
 		(descr "Mounting Hole 3.2mm, M3, no annular, generated by kicad-footprint-generator mountinghole.py")
 		(tags "mountinghole M3")
@@
 			(at 0 -4.15 0)
 			(layer "F.SilkS")
+			(hide yes)
 			(effects
 				(font
@@
 			(at 0 -4.15 0)
 			(layer "F.SilkS")
+			(hide yes)
 			(effects
 				(font
@@
 	(footprint "CAN_Isolation:ishikai_logo"
 		(layer "F.Cu")
-		(at 175 72.5)
+		(at 169.52 72.47)
 		(property "Reference" "G***"
 			(at 0 0 0)
@@
 			(at 0 -4.15 0)
 			(layer "F.SilkS")
+			(hide yes)
 			(effects
 				(font
@@
 	(footprint "MountingHole:MountingHole_3.2mm_M3"
 		(layer "F.Cu")
-		(at 148.657095 122.794905)
+		(at 143.657095 122.794905)
 		(descr "Mounting Hole 3.2mm, M3, no annular, generated by kicad-footprint-generator mountinghole.py")
 		(tags "mountinghole M3")
@@
 			(at 0 -4.15 0)
 			(layer "F.SilkS")
+			(hide yes)
 			(effects
 				(font
@@
 			(at 0 -4.15 0)
 			(layer "F.SilkS")
+			(hide yes)
 			(effects
 				(font
@@
 			(at 0 -4.15 0)
 			(layer "F.SilkS")
+			(hide yes)
 			(effects
 				(font
@@
 	)
 	(segment
-		(start 148.073695 117.24017)
-		(end 145.01896 120.294905)
-		(width 0.4)
-		(layer "F.Cu")
-		(net 3)
-	)
-	(segment
 		(start 126.657095 112.794905)
 		(end 127.657095 112.794905)
@@
 	)
 	(segment
+		(start 149.277095 106.714905)
+		(end 148.073695 107.918305)
+		(width 0.4)
+		(layer "F.Cu")
+		(net 3)
+	)
+	(segment
+		(start 131.537789 120.294905)
+		(end 131.432095 120.294905)
+		(width 0.4)
+		(layer "F.Cu")
+		(net 3)
+	)
+	(segment
 		(start 127.657095 110.794905)
 		(end 127.657095 111.794905)
@@
 	)
 	(segment
-		(start 149.277095 106.714905)
-		(end 148.073695 107.918305)
+		(start 148.073695 107.918305)
+		(end 148.073695 109.855)
 		(width 0.4)
 		(layer "F.Cu")
@@
 	)
 	(segment
+		(start 148.073695 109.855)
+		(end 147.33719 110.591505)
+		(width 0.4)
+		(layer "F.Cu")
+		(net 3)
+	)
+	(segment
 		(start 129.882095 100.294905)
 		(end 129.882095 100.569905)
@@
 	)
 	(segment
-		(start 148.073695 107.918305)
-		(end 148.073695 117.24017)
-		(width 0.4)
-		(layer "F.Cu")
-		(net 3)
-	)
-	(segment
 		(start 127.311395 110.449205)
 		(end 127.657095 110.794905)
@@
 	)
 	(segment
-		(start 145.01896 120.294905)
-		(end 131.432095 120.294905)
+		(start 136.07863 110.591505)
+		(end 135.373695 111.29644)
 		(width 0.4)
 		(layer "F.Cu")
@@
 	)
 	(segment
+		(start 135.373695 111.29644)
+		(end 135.373695 116.459)
+		(width 0.4)
+		(layer "F.Cu")
+		(net 3)
+	)
+	(segment
 		(start 126.657095 113.794905)
 		(end 126.657095 112.794905)
@@
 	)
 	(segment
+		(start 135.373695 116.459)
+		(end 131.537789 120.294905)
+		(width 0.4)
+		(layer "F.Cu")
+		(net 3)
+	)
+	(segment
 		(start 127.657095 111.794905)
 		(end 127.657095 112.794905)
@@
 	)
 	(segment
+		(start 147.33719 110.591505)
+		(end 136.07863 110.591505)
+		(width 0.4)
+		(layer "F.Cu")
+		(net 3)
+	)
+	(segment
 		(start 132.682894 86.394905)
 		(end 132.357894 86.069905)
@@
 		(polygon
 			(pts
-				(xy 143.657095 67.794905) (xy 153.657095 67.794905) (xy 153.657095 77.794905) (xy 143.657095 77.794905)
+				(xy 138.65 67.7731) (xy 148.65 67.7731) (xy 148.65 77.7731) (xy 138.65 77.7731)
 			)
 		)
@@
 		(polygon
 			(pts
-				(xy 143.657095 117.794905) (xy 153.657095 117.794905) (xy 153.657095 127.794905) (xy 143.657095 127.794905)
+				(xy 138.637 117.794905) (xy 148.637 117.794905) (xy 148.637 127.794905) (xy 138.637 127.794905)
 			)
 		)
